File: docs/filter-design/bcm-machina-noise.kicad_sch (KiCad schematic)
At the start: 14 parts, among them Q3 J113, Q4 J113, U4 4069, U5 4069

Commit message: updating filter design calculations for resonance
Parts:
- added R1: Rqf, Resistor_THT:R_Axial_DIN0207_L6.3mm_D2.5mm_P10.16mm_Horizontal, symbol Device:R
- added R2: Rqmax, Resistor_THT:R_Axial_DIN0207_L6.3mm_D2.5mm_P10.16mm_Horizontal, symbol Device:R
- RV7: value VRres -> VRq
Connections:
- net Vbp: now also R2.2; no longer RV7.3
- net at R27.1, U4.8: now also R1.2; no longer RV7.1
- net at RV7.2, U4.9: now also RV7.1, R1.1
- new net: R2.1, RV7.3
Other:
- moved on the sheet: U4D
