File: hardware/yorick/Yorick.kicad_sch (KiCad schematic)
At the start: 71 parts, among them J1 Conn_01x12, J2 AVR-ISP-6, J3 AudioJack2_SwitchT, J4 USB_C_Receptacle_USB2.0_16P, J5 AudioJack2_SwitchT, Q1 J113, Q2 J113, SW1 SW_Push, SW2 SW_Push, U1 4069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

Commit message: Renaming "kicad" folder to "hardware"
moving gerbers folder and backplate into there as well
Parts:
- J1: footprint Yorick:TEETH -> Yorick:Teeth_Pads
Changed lines of the file:
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@@
 			)
 		)
-		(property "Footprint" "Yorick:TEETH"
+		(property "Footprint" "Yorick:Teeth_Pads"
 			(at 359.41 125.73 0)
 			(effects
